File: Modello fisico/Word_Clock/_saved_circuit.sch (KiCad schematic (older format))
At the start: 425 parts

Commit message: Aggiornato svg del circuito elettrico
Connections:
- net at U?.10 (B): now also U?.10 (B)
- net at U?.11 (A): now also U?.11 (A)
- net at U?.9 (C): now also U?.9 (C)
