File: Modello fisico/Word_Clock/circuit.sch (KiCad schematic (older format))
At the start: 425 parts

Commit message: Aggiornato use case
Parts:
- removed U? (x5): 4053, symbol 4053
- added U? (x5): 4051, symbol 4051
- D? (x195): symbol LED -> LED-RESCUE-circuit
Connections:
- net VDD: now also U?.16 (VDD), U?.16 (VDD), U?.16 (VDD), U?.16 (VDD), U?.16 (VDD)
- net VSS: now also U?.8 (VSS), U?.8 (VSS), U?.8 (VSS), U?.8 (VSS), U?.8 (VSS)
- net at Q?.2 (G): now also U?.13 (X0) (x4)
- net at Q?.2 (G): now also U?.12 (X3) (x4)
- net at Q?.2 (G): now also U?.14 (X1) (x4)
- net at Q?.2 (G): now also U?.15 (X2) (x4)
- net at Q?.2 (G): now also U?.1 (X4) (x4)
- net at Q?.2 (G): now also U?.5 (X5) (x3)
- net at Q?.2 (G): now also U?.2 (X6) (x3)
- net at Q?.2 (G): now also U?.4 (X7) (x2)

Commit message: Matrice doc
Parts:
- removed IC?: ATMEGA328P-A, TQFP32, symbol ATMEGA328P-A
- removed IC?: ATMEGA328P-M, MLF/QFN32, symbol ATMEGA328P-M
- removed U?: 4051, symbol 4051
Connections:
- net labels added: Colonna_Controllata_Diretta, Dato_del_demux, Selettori_Demux_Colonne_1, Selettori_Demux_Colonne_2
- wire segments 559 -> 220
